Commit message: Melodic hardware enablement

File: description/urdf/svh-standalone.urdf.xacro (robot description, xacro)
@@ -3,5 +3,8 @@
  <xacro:include filename="$(find schunk_svh_driver)/description/urdf/svh.urdf.xacro" />
  <link name="base_link" />
- <xacro:svh parent="base_link" name="left_hand" side="-1">
+ <!-- <xacro:svh parent="base_link" name="left_hand" side="-1">
+    <origin xyz="0 0 0"  rpy= "0 0 0" /> -->
+  <!-- </xacro:svh> -->
+<xacro:svh parent="base_link" name="right_hand" side="1">
     <origin xyz="0 0 0"  rpy= "0 0 0" />
   </xacro:svh>

Commit message: backup

File: description/urdf/svh-standalone.urdf.xacro (robot description, xacro)
@@ -1,11 +1,16 @@
 <?xml version="1.0"?>
 <robot name="svh" xmlns:xacro="http://www.ros.org/wiki/xacro">
+ <xacro:property name="left_right" default="right_hand"/>
  <xacro:include filename="$(find schunk_svh_driver)/description/urdf/svh.urdf.xacro" />
  <link name="base_link" />
- <!-- <xacro:svh parent="base_link" name="left_hand" side="-1">
-    <origin xyz="0 0 0"  rpy= "0 0 0" /> -->
-  <!-- </xacro:svh> -->
-<xacro:svh parent="base_link" name="right_hand" side="1">
-    <origin xyz="0 0 0"  rpy= "0 0 0" />
+ <xacro:if value="${left_right == 'left_hand'}">
+  <xacro:svh parent="base_link" name="left_hand" side="-1">
+   <origin xyz="0 0 0"  rpy= "0 0 0" /> -->
   </xacro:svh>
+ </xacro:if>
+ <xacro:if value="${left_right == 'right_hand'}">
+  <xacro:svh parent="base_link" name="right_hand" side="1">
+   <origin xyz="0 0 0"  rpy= "0 0 0" />
+  </xacro:svh>
+ </xacro:if>
 </robot>
